Commit message: add axis print torque data

File: TECObot_urdf_test_MESH_3/urdf/TECObot_urdf_test_MESH_3.urdf (robot description, URDF)
Before this commit: robot TECObot_urdf_test_MESH_3, 3 links, 2 joints
Links:
- link base_link: mass 0.726077498939582 -> 0.72608
- link link_1: mass 0.706624909903978 -> 0.70662
- link link_2: mass 0.706624392841053 -> 0.70662
Joints:
- joint joint_1: origin xyz=0 0 0 rpy=0 0 0 -> xyz=0 0 0.1296 rpy=0 0 0
- joint joint_2: axis -1 0 0 -> -0.99321 0.11637 0; origin xyz=0.091378 -0.06328 0.1301 rpy=0 0 2.5359 -> xyz=-0.11015 0.012905 0.1296 rpy=0 0 0
