Commit message: ros dynamics data topic test ok

File: test/urdf/test.urdf (robot description, URDF)
Before this commit: robot test, 2 links, 1 joints
Links:
- added link 2, mass 0.70663; collision mesh filename=package://test/meshes/2.STL; visual mesh filename=package://test/meshes/2.STL
- link 1: mass 0.084627 -> 0.70663
- link base_link: mass 0.56321 -> 0.72607
Joints:
- removed joint aa
- added joint j1: type revolute, parent base_link, child 1, origin xyz=0 0 0 rpy=0 0 0, axis 0 0 1, limit lower=-2.5 upper=2.5 effort=1000 velocity=0.5
- added joint j2: type revolute, parent 1, child 2, origin xyz=0.0049033 0.11079 0.1296 rpy=0 0 0, axis 0.044214 0.99902 0, limit lower=-2.5 upper=2.5 effort=1000 velocity=0.5
