Commit message: j3,j4 fixed length ok on URDF

File: dynamics/src/dynamics/urdf/random.urdf (robot description, URDF)
Before this commit: robot tecobot, 8 links, 7 joints
Links:
- link 2: mass 1.8060602894988051 -> 1.81432701922486
- link 3: mass 0.44484587990482194 -> 0.44267362700812
Joints:
- joint j2: origin xyz=0 0.11115 0 rpy=-1.5708 0 3.1416 -> xyz=0 0.11115 -6.411407844118837e-06 rpy=-1.5708 0 3.1416

Commit message: add combox select arm design parameter

File: dynamics/src/dynamics/urdf/random.urdf (robot description, URDF)
Before this commit: robot tecobot, 8 links, 7 joints
Links:
- link 2: mass 1.81432701922486 -> 1.8060602894988051
- link 3: mass 0.44267362700812 -> 0.44484587990482194
Joints:
- joint j3: origin xyz=0 0.408000000000056 0 rpy=0 0 0 -> xyz=0 0.32650000000005597 0 rpy=0 0 0
- joint j4: origin xyz=0 0.372499999999936 0.0109000000011954 rpy=1.57079632675385 0 -3.14159265356591 -> xyz=0 0.307499999999936 0.0109000000011954 rpy=1.57079632675385 0 -3.14159265356591

Commit message: fixed write mesh name

File: dynamics/src/dynamics/urdf/random.urdf (robot description, URDF)
Before this commit: robot tecobot, 8 links, 7 joints
Links:
- link 2: mass 1.8060602894988051 -> 1.616589494712605; geometry collision mesh filename=package://tecobot/meshes/2.STL; visual mesh filename=package://dynamics/src/dynamics/meshes/random_2_25.0.STL
- link 3: mass 0.44484587990482194 -> 0.5453617078222979; geometry collision mesh filename=package://tecobot/meshes/3.STL; visual mesh filename=package://dynamics/src/dynamics/meshes/random_3_45.0.STL
Joints:
- joint j3: origin xyz=0 0.32650000000005597 0 rpy=0 0 0 -> xyz=0 0.25 0 rpy=0 0 0
- joint j4: origin xyz=0 0.307499999999936 0.0109000000011954 rpy=1.57079632675385 0 -3.14159265356591 -> xyz=0 0.45000000000000007 0.0109000000011954 rpy=1.57079632675385 0 -3.14159265356591

Commit message: arm data rebuild & fixed random arm stl

File: dynamics/src/dynamics/urdf/random.urdf (robot description, URDF)
Before this commit: robot tecobot, 8 links, 7 joints
Links:
- link 2: mass 1.616589494712605 -> 1.775166295877986; geometry collision mesh filename=package://tecobot/meshes/2.STL; visual mesh filename=package://dynamics/src/dynamics/meshes/random_2_40.0.STL
- link 3: mass 0.5453617078222979 -> 0.45737171513244773; geometry collision mesh filename=package://tecobot/meshes/3.STL; visual mesh filename=package://dynamics/src/dynamics/meshes/random_3_20.0.STL
Joints:
- joint j3: origin xyz=0 0.25 0 rpy=0 0 0 -> xyz=0 0.4 0 rpy=0 0 0
- joint j4: origin xyz=0 0.45000000000000007 0.0109000000011954 rpy=1.57079632675385 0 -3.14159265356591 -> xyz=0 0.20000000000000004 0.0203999999999699 rpy=1.57079632675385 0 -3.14159265356591

Commit message: add GUI progress item

File: dynamics/src/dynamics/urdf/random.urdf (robot description, URDF)
Before this commit: robot tecobot, 8 links, 7 joints
Links:
- link 2: mass 1.775166295877986 -> 1.5633927364282878; geometry collision mesh filename=package://tecobot/meshes/2.STL; visual mesh filename=package://dynamics/src/dynamics/meshes/random_2_20.0.STL
Joints:
- joint j3: origin xyz=0 0.4 0 rpy=0 0 0 -> xyz=0 0.19999999999999998 0 rpy=0 0 0

Commit message: add motor size and data & add trajectory generate

File: dynamics/src/dynamics/urdf/random.urdf (robot description, URDF)
Before this commit: robot tecobot, 8 links, 7 joints
Links:
- link 2: mass 1.5633927364282878 -> 1.775166295877986; geometry collision mesh filename=package://tecobot/meshes/2.STL; visual mesh filename=package://dynamics/src/dynamics/meshes/random_2_40.0.STL
- link 3: mass 0.45737171513244773 -> 0.5105337194421253; geometry collision mesh filename=package://tecobot/meshes/3.STL; visual mesh filename=package://dynamics/src/dynamics/meshes/random_3_35.0.STL
Joints:
- joint j3: origin xyz=0 0.19999999999999998 0 rpy=0 0 0 -> xyz=0 0.4 0 rpy=0 0 0
- joint j4: origin xyz=0 0.20000000000000004 0.0203999999999699 rpy=1.57079632675385 0 -3.14159265356591 -> xyz=0 0.35000000000000003 0.0203999999999699 rpy=1.57079632675385 0 -3.14159265356591

Commit message: add matlab optimatal trajectory random arm

File: dynamics/src/dynamics/urdf/random.urdf (robot description, URDF)
Before this commit: robot tecobot, 8 links, 7 joints
Links:
- link 2: mass 1.775166295877986 -> 1.5633927364282878; geometry collision mesh filename=package://tecobot/meshes/2.STL; visual mesh filename=package://dynamics/src/dynamics/meshes/random_2_20.0.STL
- link 3: mass 0.5105337194421253 -> 0.45737171513244773; geometry collision mesh filename=package://tecobot/meshes/3.STL; visual mesh filename=package://dynamics/src/dynamics/meshes/random_3_20.0.STL
Joints:
- joint j3: origin xyz=0 0.4 0 rpy=0 0 0 -> xyz=0 0.19999999999999998 0 rpy=0 0 0
- joint j4: origin xyz=0 0.35000000000000003 0.0203999999999699 rpy=1.57079632675385 0 -3.14159265356591 -> xyz=0 0.20000000000000004 0.0203999999999699 rpy=1.57079632675385 0 -3.14159265356591

Commit message: add random axis robot urdf function

File: dynamics/src/dynamics/urdf/random.urdf (robot description, URDF)
Before this commit: robot tecobot, 8 links, 7 joints
Links:
- link 2: mass 1.5633927364282878 -> 1.7281655242126162; geometry collision mesh filename=package://tecobot/meshes/2.STL; visual mesh filename=package://dynamics/src/dynamics/meshes/random_2_35.0.STL
- link 3: mass 0.45737171513244773 -> 0.5468457974291466; geometry collision mesh filename=package://tecobot/meshes/3.STL; visual mesh filename=package://dynamics/src/dynamics/meshes/random_3_35.0.STL
Joints:
- joint j3: origin xyz=0 0.19999999999999998 0 rpy=0 0 0 -> xyz=0 0.3670951094329047 0 rpy=0 0 0
- joint j4: origin xyz=0 0.20000000000000004 0.0203999999999699 rpy=1.57079632675385 0 -3.14159265356591 -> xyz=0 0.45642114554254 0.0203999999999699 rpy=1.57079632675385 0 -3.14159265356591

Commit message: add robot worksapce input

File: dynamics/src/dynamics/urdf/random.urdf (robot description, URDF)
Before this commit: robot tecobot, 8 links, 7 joints
Links:
- link 2: mass 1.7281655242126162 -> 1.5633927364282878; geometry collision mesh filename=package://tecobot/meshes/2.STL; visual mesh filename=package://dynamics/src/dynamics/meshes/random_2_20.0.STL
- link 3: mass 0.5468457974291466 -> 0.45737171513244773; geometry collision mesh filename=package://tecobot/meshes/3.STL; visual mesh filename=package://dynamics/src/dynamics/meshes/random_3_20.0.STL
Joints:
- joint j3: origin xyz=0 0.3670951094329047 0 rpy=0 0 0 -> xyz=0 0.19999999999999998 0 rpy=0 0 0
- joint j4: origin xyz=0 0.45642114554254 0.0203999999999699 rpy=1.57079632675385 0 -3.14159265356591 -> xyz=0 0.20000000000000004 0.0203999999999699 rpy=1.57079632675385 0 -3.14159265356591

Commit message: complete connect optimal method input data

File: dynamics/src/dynamics/urdf/random.urdf (robot description, URDF)
Before this commit: robot tecobot, 8 links, 7 joints
Links:
- link 2: mass 1.5633927364282878 -> 1.7316962465750905; geometry collision mesh filename=package://tecobot/meshes/2.STL; visual mesh filename=package://dynamics/src/dynamics/meshes/random_2_35.0.STL
- link 3: mass 0.45737171513244773 -> 0.4976182768428218; geometry collision mesh filename=package://tecobot/meshes/3.STL; visual mesh filename=package://dynamics/src/dynamics/meshes/random_3_35.0.STL
Joints:
- joint j3: origin xyz=0 0.19999999999999998 0 rpy=0 0 0 -> xyz=0 0.37744272761497305 0 rpy=0 0 0
- joint j4: origin xyz=0 0.20000000000000004 0.0203999999999699 rpy=1.57079632675385 0 -3.14159265356591 -> xyz=0 0.312148236267336 0.0203999999999699 rpy=1.57079632675385 0 -3.14159265356591

Commit message: fix static dynamic space scan

File: dynamics/src/dynamics/urdf/random.urdf (robot description, URDF)
Before this commit: robot tecobot, 8 links, 7 joints
Links:
- link 2: mass 1.7316962465750905 -> 1.775166295877986; geometry collision mesh filename=package://tecobot/meshes/2.STL; visual mesh filename=package://dynamics/src/dynamics/meshes/random_2_40.0.STL
- link 3: mass 0.4976182768428218 -> 0.5276892469859136; geometry collision mesh filename=package://tecobot/meshes/3.STL; visual mesh filename=package://dynamics/src/dynamics/meshes/random_3_40.0.STL
Joints:
- joint j3: origin xyz=0 0.37744272761497305 0 rpy=0 0 0 -> xyz=0 0.4 0 rpy=0 0 0
- joint j4: origin xyz=0 0.312148236267336 0.0203999999999699 rpy=1.57079632675385 0 -3.14159265356591 -> xyz=0 0.4 0.0203999999999699 rpy=1.57079632675385 0 -3.14159265356591

Commit message: add CJM select function

File: dynamics/src/dynamics/urdf/random.urdf (robot description, URDF)
Before this commit: robot tecobot, 8 links, 7 joints
Links:
- link 2: mass 1.775166295877986 -> 1.828869841797684; geometry collision mesh filename=package://tecobot/meshes/2.STL; visual mesh filename=package://dynamics/src/dynamics/meshes/random_2_45.0.STL
- link 3: mass 0.5276892469859136 -> 0.5457872554801146; geometry collision mesh filename=package://tecobot/meshes/3.STL; visual mesh filename=package://dynamics/src/dynamics/meshes/random_3_45.0.STL
Joints:
- joint j3: origin xyz=0 0.4 0 rpy=0 0 0 -> xyz=0 0.45 0 rpy=0 0 0
- joint j4: origin xyz=0 0.4 0.0203999999999699 rpy=1.57079632675385 0 -3.14159265356591 -> xyz=0 0.45000000000000007 0.0203999999999699 rpy=1.57079632675385 0 -3.14159265356591

Commit message: add motor module select output excel

File: dynamics/src/dynamics/urdf/random.urdf (robot description, URDF)
Before this commit: robot tecobot, 8 links, 7 joints
Links:
- link 2: mass 1.828869841797684 -> 1.5633927364282878; geometry collision mesh filename=package://tecobot/meshes/2.STL; visual mesh filename=package://dynamics/src/dynamics/meshes/random_2_20.0.STL
- link 3: mass 0.5457872554801146 -> 0.45737171513244773; geometry collision mesh filename=package://tecobot/meshes/3.STL; visual mesh filename=package://dynamics/src/dynamics/meshes/random_3_20.0.STL
Joints:
- joint j3: origin xyz=0 0.45 0 rpy=0 0 0 -> xyz=0 0.19999999999999998 0 rpy=0 0 0
- joint j4: origin xyz=0 0.45000000000000007 0.0203999999999699 rpy=1.57079632675385 0 -3.14159265356591 -> xyz=0 0.20000000000000004 0.0203999999999699 rpy=1.57079632675385 0 -3.14159265356591

Commit message: arm workspace plane test ok

File: dynamics/src/dynamics/urdf/random.urdf (robot description, URDF)
Before this commit: robot tecobot, 8 links, 7 joints
Links:
- link 2: mass 1.5633927364282878 -> 1.775166295877986; geometry collision mesh filename=package://tecobot/meshes/2.STL; visual mesh filename=package://dynamics/src/dynamics/meshes/random_2_40.0.STL
- link 3: mass 0.45737171513244773 -> 0.49206838913812917; geometry collision mesh filename=package://tecobot/meshes/3.STL; visual mesh filename=package://dynamics/src/dynamics/meshes/random_3_30.0.STL
Joints:
- joint j3: origin xyz=0 0.19999999999999998 0 rpy=0 0 0 -> xyz=0 0.4 0 rpy=0 0 0
- joint j4: origin xyz=0 0.20000000000000004 0.0203999999999699 rpy=1.57079632675385 0 -3.14159265356591 -> xyz=0 0.30000000000000004 0.0203999999999699 rpy=1.57079632675385 0 -3.14159265356591

Commit message: GUI set the joint angle limit ok

File: dynamics/src/dynamics/urdf/random.urdf (robot description, URDF)
Before this commit: robot tecobot, 8 links, 7 joints
Links:
- link 2: mass 1.775166295877986 -> 1.5633927364282878; geometry collision mesh filename=package://tecobot/meshes/2.STL; visual mesh filename=package://dynamics/src/dynamics/meshes/random_2_20.0.STL
- link 3: mass 0.49206838913812917 -> 0.45737171513244773; geometry collision mesh filename=package://tecobot/meshes/3.STL; visual mesh filename=package://dynamics/src/dynamics/meshes/random_3_20.0.STL
Joints:
- joint j3: origin xyz=0 0.4 0 rpy=0 0 0 -> xyz=0 0.19999999999999998 0 rpy=0 0 0
- joint j4: origin xyz=0 0.30000000000000004 0.0203999999999699 rpy=1.57079632675385 0 -3.14159265356591 -> xyz=0 0.20000000000000004 0.0203999999999699 rpy=1.57079632675385 0 -3.14159265356591

Commit message: add can input axis length information

File: dynamics/src/dynamics/urdf/random.urdf (robot description, URDF)
Before this commit: robot tecobot, 8 links, 7 joints
Links:
- link 2: mass 1.5633927364282878 -> 1.7100488825938092; geometry collision mesh filename=package://tecobot/meshes/2.STL; visual mesh filename=package://dynamics/src/dynamics/meshes/random_2_31.4.STL
- link 3: mass 0.45737171513244773 -> 0.4880137856928178; geometry collision mesh filename=package://tecobot/meshes/3.STL; visual mesh filename=package://dynamics/src/dynamics/meshes/random_3_28.4.STL
Joints:
- joint j3: origin xyz=0 0.19999999999999998 0 rpy=0 0 0 -> xyz=0 0.314 0 rpy=0 0 0
- joint j4: origin xyz=0 0.20000000000000004 0.0203999999999699 rpy=1.57079632675385 0 -3.14159265356591 -> xyz=0 0.28400000000000003 0.0203999999999699 rpy=1.57079632675385 0 -3.14159265356591

Commit message: add interface unit

File: dynamics/src/dynamics/urdf/random.urdf (robot description, URDF)
Before this commit: robot tecobot, 8 links, 7 joints
Links:
- link 2: mass 1.7100488825938092 -> 1.7735141504327667; geometry collision mesh filename=package://tecobot/meshes/2.STL; visual mesh filename=package://dynamics/src/dynamics/meshes/random_2_50.0.STL
- link 3: mass 0.4880137856928178 -> 0.5617153870541877; geometry collision mesh filename=package://tecobot/meshes/3.STL; visual mesh filename=package://dynamics/src/dynamics/meshes/random_3_50.0.STL
Joints:
- joint j3: origin xyz=0 0.314 0 rpy=0 0 0 -> xyz=0 0.5 0 rpy=0 0 0
- joint j4: origin xyz=0 0.28400000000000003 0.0203999999999699 rpy=1.57079632675385 0 -3.14159265356591 -> xyz=0 0.5 0.0203999999999699 rpy=1.57079632675385 0 -3.14159265356591

Commit message: interface add joint 7

File: dynamics/src/dynamics/urdf/random.urdf (robot description, URDF)
Before this commit: robot tecobot, 8 links, 7 joints
Links:
- link 2: mass 1.7735141504327667 -> 1.6711508152086418; geometry collision mesh filename=package://tecobot/meshes/2.STL; visual mesh filename=package://dynamics/src/dynamics/meshes/random_2_20.0.STL
- link 3: mass 0.5617153870541877 -> 0.4593520518300629; geometry collision mesh filename=package://tecobot/meshes/3.STL; visual mesh filename=package://dynamics/src/dynamics/meshes/random_3_20.0.STL
Joints:
- joint j3: origin xyz=0 0.5 0 rpy=0 0 0 -> xyz=0 0.19999999999999998 0 rpy=0 0 0
- joint j4: origin xyz=0 0.5 0.0203999999999699 rpy=1.57079632675385 0 -3.14159265356591 -> xyz=0 0.20000000000000004 0.0203999999999699 rpy=1.57079632675385 0 -3.14159265356591

Commit message: add 7 dof single arm todo fix dh

File: dynamics/src/dynamics/urdf/random.urdf (robot description, URDF)
Before this commit: robot tecobot, 8 links, 7 joints
Links:
- link 2: mass 1.6711508152086418 -> 1.6029085917258918; geometry collision mesh filename=package://tecobot/meshes/2.STL; visual mesh filename=package://dynamics/src/dynamics/meshes/random_2_0.0.STL
- link 3: mass 0.4593520518300629 -> 0.39110982834731295; geometry collision mesh filename=package://tecobot/meshes/3.STL; visual mesh filename=package://dynamics/src/dynamics/meshes/random_3_0.0.STL
Joints:
- joint j3: origin xyz=0 0.19999999999999998 0 rpy=0 0 0 -> xyz=0 0.0 0 rpy=0 0 0
- joint j4: origin xyz=0 0.20000000000000004 0.0203999999999699 rpy=1.57079632675385 0 -3.14159265356591 -> xyz=0 0.0 0.0203999999999699 rpy=1.57079632675385 0 -3.14159265356591

Commit message: add select sturcture function

File: dynamics/src/dynamics/urdf/random.urdf (robot description, URDF)
Before this commit: robot tecobot, 8 links, 7 joints
Links:
- link 2: mass 1.6029085917258918 -> 1.701395206086981; geometry collision mesh filename=package://tecobot/meshes/2.STL; visual mesh filename=package://dynamics/src/dynamics/meshes/random_2_35.0.STL
- link 3: mass 0.39110982834731295 -> 0.4903996894016639; geometry collision mesh filename=package://tecobot/meshes/3.STL; visual mesh filename=package://dynamics/src/dynamics/meshes/random_3_35.0.STL
Joints:
- joint j3: origin xyz=0 0.0 0 rpy=0 0 0 -> xyz=0 0.2886383512576618 0 rpy=0 0 0
- joint j4: origin xyz=0 0.0 0.0203999999999699 rpy=1.57079632675385 0 -3.14159265356591 -> xyz=0 0.2909924559519933 0.0203999999999699 rpy=1.57079632675385 0 -3.14159265356591

Commit message: fixed dynamics general robot

File: dynamics/src/dynamics/urdf/random.urdf (robot description, URDF)
Before this commit: robot tecobot, 8 links, 7 joints
Links:
- link 2: mass 1.701395206086981 -> 1.6711508152086418; geometry collision mesh filename=package://tecobot/meshes/2.STL; visual mesh filename=package://dynamics/src/dynamics/meshes/random_2_20.0.STL
- link 3: mass 0.4903996894016639 -> 0.4593520518300629; geometry collision mesh filename=package://tecobot/meshes/3.STL; visual mesh filename=package://dynamics/src/dynamics/meshes/random_3_20.0.STL
Joints:
- joint j3: origin xyz=0 0.2886383512576618 0 rpy=0 0 0 -> xyz=0 0.19999999999999998 0 rpy=0 0 0
- joint j4: origin xyz=0 0.2909924559519933 0.0203999999999699 rpy=1.57079632675385 0 -3.14159265356591 -> xyz=0 0.20000000000000004 0.0203999999999699 rpy=1.57079632675385 0 -3.14159265356591

Commit message: build robotoptenv environment

File: dynamics/src/dynamics/urdf/random.urdf (robot description, URDF)
Before this commit: robot tecobot, 8 links, 7 joints
Links:
- link 2: mass 1.6029085917258918 -> 1.7223324828207043; geometry collision mesh filename=package://tecobot/meshes/2.STL; visual mesh filename=package://dynamics/src/dynamics/meshes/random_2_35.0.STL
- link 3: mass 0.39110982834731295 -> 0.5071216082679878; geometry collision mesh filename=package://tecobot/meshes/3.STL; visual mesh filename=package://dynamics/src/dynamics/meshes/random_3_35.0.STL
Joints:
- joint j3: origin xyz=0 0.0 0 rpy=0 0 0 -> xyz=0 0.35 0 rpy=0 0 0
- joint j4: origin xyz=0 0.0 0.0203999999999699 rpy=1.57079632675385 0 -3.14159265356591 -> xyz=0 0.34 0.0203999999999699 rpy=1.57079632675385 0 -3.14159265356591

Commit message: run drl ok but have agent mat1 mat2 bug

File: dynamics/src/dynamics/urdf/random.urdf (robot description, URDF)
Before this commit: robot tecobot, 8 links, 7 joints
Links:
- link 2: mass 1.7223324828207043 -> 1.8349321515674326; geometry collision mesh filename=package://tecobot/meshes/2.STL; visual mesh filename=package://dynamics/src/dynamics/meshes/random_2_68.00000000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
- link 3: mass 0.5071216082679878 -> 0.5702582541101929; geometry collision mesh filename=package://tecobot/meshes/3.STL; visual mesh filename=package://dynamics/src/dynamics/meshes/random_3_52.50368953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
Joints:
- joint j3: origin xyz=0 0.35 0 rpy=0 0 0 -> xyz=0 0.6800000000005599 0 rpy=0 0 0
- joint j4: origin xyz=0 0.34 0.0203999999999699 rpy=1.57079632675385 0 -3.14159265356591 -> xyz=0 0.5250368953999999 0.0203999999999699 rpy=1.57079632675385 0 -3.14159265356591

Commit message: succsess run drl test only consider torque

File: dynamics/src/dynamics/urdf/random.urdf (robot description, URDF)
Before this commit: robot tecobot, 8 links, 7 joints
Links:
- link 2: mass 1.8349321515674326 -> 1.7325688163431168; geometry collision mesh filename=package://tecobot/meshes/2.STL; visual mesh filename=package://dynamics/src/dynamics/meshes/random_2_35.0.STL
- link 3: mass 0.5702582541101929 -> 0.5139458306162629; geometry collision mesh filename=package://tecobot/meshes/3.STL; visual mesh filename=package://dynamics/src/dynamics/meshes/random_3_35.0.STL
Joints:
- joint j3: origin xyz=0 0.6800000000005599 0 rpy=0 0 0 -> xyz=0 0.38 0 rpy=0 0 0
- joint j4: origin xyz=0 0.5250368953999999 0.0203999999999699 rpy=1.57079632675385 0 -3.14159265356591 -> xyz=0 0.36000000000000004 0.0203999999999699 rpy=1.57079632675385 0 -3.14159265356591

Commit message: fix reward v1

File: dynamics/src/dynamics/urdf/random.urdf (robot description, URDF)
Before this commit: robot tecobot, 8 links, 7 joints
Links:
- link 2: mass 1.7325688163431168 -> 1.7257445939948417
Joints:
- joint j3: origin xyz=0 0.38 0 rpy=0 0 0 -> xyz=0 0.36 0 rpy=0 0 0

Commit message: fix tensorboard output ok

File: dynamics/src/dynamics/urdf/random.urdf (robot description, URDF)
Before this commit: robot tecobot, 8 links, 7 joints
Links:
- link 2: mass 1.7257445939948417 -> 1.831520040393104
- link 3: mass 0.5139458306162629 -> 0.46617627417833785
Joints:
- joint j3: origin xyz=0 0.36 0 rpy=0 0 0 -> xyz=0 0.6699999999999999 0 rpy=0 0 0
- joint j4: origin xyz=0 0.36000000000000004 0.0203999999999699 rpy=1.57079632675385 0 -3.14159265356591 -> xyz=0 0.22000000000000003 0.0203999999999699 rpy=1.57079632675385 0 -3.14159265356591

Commit message: add 0718 train result

File: dynamics/src/dynamics/urdf/random.urdf (robot description, URDF)
Before this commit: robot tecobot, 8 links, 7 joints
Links:
- link 2: mass 1.831520040393104 -> 1.575611702332792
- link 3: mass 0.46617627417833785 -> 0.21368004729216314
Joints:
- joint j3: origin xyz=0 0.6699999999999999 0 rpy=0 0 0 -> xyz=0 -0.08000000000000002 0 rpy=0 0 0
- joint j4: origin xyz=0 0.22000000000000003 0.0203999999999699 rpy=1.57079632675385 0 -3.14159265356591 -> xyz=0 -0.52 0.0203999999999699 rpy=1.57079632675385 0 -3.14159265356591

Commit message: add episode truncates not test

File: dynamics/src/dynamics/urdf/random.urdf (robot description, URDF)
Before this commit: robot tecobot, 8 links, 7 joints
Links:
- link 2: mass 1.575611702332792 -> 1.7735141504327667
- link 3: mass 0.21368004729216314 -> 0.41840671774041294
Joints:
- joint j3: origin xyz=0 -0.08000000000000002 0 rpy=0 0 0 -> xyz=0 0.5 0 rpy=0 0 0
- joint j4: origin xyz=0 -0.52 0.0203999999999699 rpy=1.57079632675385 0 -3.14159265356591 -> xyz=0 0.08000000000000002 0.0203999999999699 rpy=1.57079632675385 0 -3.14159265356591

Commit message: TODO: 修正 state 為 1*7 的 numpy array, 因新增可達半徑判斷

File: dynamics/src/dynamics/urdf/random.urdf (robot description, URDF)
Before this commit: robot tecobot, 8 links, 7 joints
Links:
- link 2: mass 1.7735141504327667 -> 1.7086840381241541
- link 3: mass 0.41840671774041294 -> 0.5173579417904003
Joints:
- joint j3: origin xyz=0 0.5 0 rpy=0 0 0 -> xyz=0 0.31 0 rpy=0 0 0
- joint j4: origin xyz=0 0.08000000000000002 0.0203999999999699 rpy=1.57079632675385 0 -3.14159265356591 -> xyz=0 0.37000000000000005 0.0203999999999699 rpy=1.57079632675385 0 -3.14159265356591

Commit message: fixed  修正 state 為 1*7 的 numpy array, 因新增可達半徑判斷

File: dynamics/src/dynamics/urdf/random.urdf (robot description, URDF)
Before this commit: robot tecobot, 8 links, 7 joints
Links:
- link 2: mass 1.7086840381241541 -> 1.7291567051689791
- link 3: mass 0.5173579417904003 -> 0.5105337194421253
Joints:
- joint j3: origin xyz=0 0.31 0 rpy=0 0 0 -> xyz=0 0.37 0 rpy=0 0 0
- joint j4: origin xyz=0 0.37000000000000005 0.0203999999999699 rpy=1.57079632675385 0 -3.14159265356591 -> xyz=0 0.35000000000000003 0.0203999999999699 rpy=1.57079632675385 0 -3.14159265356591

Commit message: fixed stl conv urdf & 重置軸長

File: dynamics/src/dynamics/urdf/random.urdf (robot description, URDF)
Before this commit: robot tecobot, 8 links, 7 joints
Links:
- link 2: mass 1.7291567051689791 -> 1.7223324828207043
- link 3: mass 0.5105337194421253 -> 0.5071216082679878
Joints:
- joint j3: origin xyz=0 0.37 0 rpy=0 0 0 -> xyz=0 0.35 0 rpy=0 0 0
- joint j4: origin xyz=0 0.35000000000000003 0.0203999999999699 rpy=1.57079632675385 0 -3.14159265356591 -> xyz=0 0.34 0.0203999999999699 rpy=1.57079632675385 0 -3.14159265356591
