Commit message: TODO: fix stl conv 6dof urdf & 修改為可調整dof的方式

File: dynamics/src/dynamics/urdf/random.urdf (robot description, URDF)
Before this commit: robot tecobot, 8 links, 7 joints
Links:
- link 2: mass 1.7223324828207043 -> 1.7325688163431168
- link 3: mass 0.5071216082679878 -> 0.5105337194421253
Joints:
- joint j3: origin xyz=0 0.35 0 rpy=0 0 0 -> xyz=0 0.38 0 rpy=0 0 0
- joint j4: origin xyz=0 0.34 0.0203999999999699 rpy=1.57079632675385 0 -3.14159265356591 -> xyz=0 0.35000000000000003 0.0203999999999699 rpy=1.57079632675385 0 -3.14159265356591

Commit message: DRL_v1 consider torque & reach_distance

File: dynamics/src/dynamics/urdf/random.urdf (robot description, URDF)
Before this commit: robot tecobot, 8 links, 7 joints
Links:
- link 2: mass 1.7325688163431168 -> 1.7462172610396667
- link 3: mass 0.5105337194421253 -> 0.5139458306162629
Joints:
- joint j3: origin xyz=0 0.38 0 rpy=0 0 0 -> xyz=0 0.35 0 rpy=0 0 0

Commit message: TODO: 向量編碼動作

File: dynamics/src/dynamics/urdf/random.urdf (robot description, URDF)
Before this commit: robot tecobot, 8 links, 7 joints
Links:
- link 2: mass 1.7462172610396667 -> 1.7086840381241541
- link 3: mass 0.5139458306162629 -> 0.5071216082679878
Joints:
- joint j3: origin xyz=0 0.35 0 rpy=0 0 0 -> xyz=0 0.31 0 rpy=0 0 0
- joint j4: origin xyz=0 0.35000000000000003 0.0203999999999699 rpy=1.57079632675385 0 -3.14159265356591 -> xyz=0 0.34 0.0203999999999699 rpy=1.57079632675385 0 -3.14159265356591

Commit message: add consider motor type & fixed reward function

File: dynamics/src/dynamics/urdf/random.urdf (robot description, URDF)
Before this commit: robot tecobot, 8 links, 7 joints
Links:
- link 2: mass 1.7086840381241541 -> 1.701859815775879
- link 3: mass 0.5071216082679878 -> 0.5446548311835002
Joints:
- joint j3: origin xyz=0 0.31 0 rpy=0 0 0 -> xyz=0 0.29 0 rpy=0 0 0
- joint j4: origin xyz=0 0.34 0.0203999999999699 rpy=1.57079632675385 0 -3.14159265356591 -> xyz=0 0.45000000000000007 0.0203999999999699 rpy=1.57079632675385 0 -3.14159265356591

Commit message: consider cost & weight

File: dynamics/src/dynamics/urdf/random.urdf (robot description, URDF)
Before this commit: robot tecobot, 8 links, 7 joints
Links:
- link 2: mass 1.701859815775879 -> 1.6540902593379543
- link 3: mass 0.5446548311835002 -> 0.5105337194421253
Joints:
- joint j3: origin xyz=0 0.29 0 rpy=0 0 0 -> xyz=0 0.14999999999999997 0 rpy=0 0 0
- joint j4: origin xyz=0 0.45000000000000007 0.0203999999999699 rpy=1.57079632675385 0 -3.14159265356591 -> xyz=0 0.35000000000000003 0.0203999999999699 rpy=1.57079632675385 0 -3.14159265356591

Commit message: add interface input optimal design data not test

File: dynamics/src/dynamics/urdf/random.urdf (robot description, URDF)
Before this commit: robot tecobot, 8 links, 7 joints
Links:
- link 2: mass 1.6540902593379543 -> 1.6952268728433366
- link 3: mass 0.5105337194421253 -> 0.46150637162178565
Joints:
- joint j3: origin xyz=0 0.14999999999999997 0 rpy=0 0 0 -> xyz=0 0.27056058963489293 0 rpy=0 0 0
- joint j4: origin xyz=0 0.35000000000000003 0.0203999999999699 rpy=1.57079632675385 0 -3.14159265356591 -> xyz=0 0.20631374442911377 0.0203999999999699 rpy=1.57079632675385 0 -3.14159265356591

Commit message: add interface input drl data

File: dynamics/src/dynamics/urdf/random.urdf (robot description, URDF)
Before this commit: robot tecobot, 8 links, 7 joints
Links:
- link 2: mass 1.6952268728433366 -> 1.7393930386913918
- link 3: mass 0.46150637162178565 -> 0.5071216082679878
Joints:
- joint j3: origin xyz=0 0.27056058963489293 0 rpy=0 0 0 -> xyz=0 0.4 0 rpy=0 0 0
- joint j4: origin xyz=0 0.20631374442911377 0.0203999999999699 rpy=1.57079632675385 0 -3.14159265356591 -> xyz=0 0.34 0.0203999999999699 rpy=1.57079632675385 0 -3.14159265356591

Commit message: fixed no module named dynamics

File: dynamics/src/dynamics/urdf/random.urdf (robot description, URDF)
Before this commit: robot tecobot, 8 links, 7 joints
Links:
- link 2: mass 1.7393930386913918 -> 1.7189203716465666
- link 3: mass 0.5071216082679878 -> 0.5105337194421253
Joints:
- joint j3: origin xyz=0 0.4 0 rpy=0 0 0 -> xyz=0 0.33999999999999997 0 rpy=0 0 0
- joint j4: origin xyz=0 0.34 0.0203999999999699 rpy=1.57079632675385 0 -3.14159265356591 -> xyz=0 0.35000000000000003 0.0203999999999699 rpy=1.57079632675385 0 -3.14159265356591

Commit message: fixed motor rated

File: dynamics/src/dynamics/urdf/random.urdf (robot description, URDF)
Before this commit: robot tecobot, 8 links, 7 joints
Links:
- link 2: mass 1.7189203716465666 -> 1.7223324828207043
- link 3: mass 0.5105337194421253 -> 0.5071216082679878
Joints:
- joint j3: origin xyz=0 0.33999999999999997 0 rpy=0 0 0 -> xyz=0 0.35 0 rpy=0 0 0

Commit message: add random axis length reset (DRL)

File: dynamics/src/dynamics/urdf/random.urdf (robot description, URDF)
Before this commit: robot tecobot, 8 links, 7 joints
Links:
- link 2: mass 1.7223324828207043 -> 1.7454142780180935
- link 3: mass 0.5071216082679878 -> 0.5518875094329906
Joints:
- joint j3: origin xyz=0 0.35 0 rpy=0 0 0 -> xyz=0 0.4176466680580058 0 rpy=0 0 0
- joint j4: origin xyz=0 0.35000000000000003 0.0203999999999699 rpy=1.57079632675385 0 -3.14159265356591 -> xyz=0 0.47119707676675754 0.0203999999999699 rpy=1.57079632675385 0 -3.14159265356591

Commit message: add ddqn alog v2

File: dynamics/src/dynamics/urdf/random.urdf (robot description, URDF)
Before this commit: robot tecobot, 8 links, 7 joints
Links:
- link 2: mass 1.7454142780180935 -> 1.7679247444870383
- link 3: mass 0.5518875094329906 -> 0.4721316268780683
Joints:
- joint j3: origin xyz=0 0.4176466680580058 0 rpy=0 0 0 -> xyz=0 0.4836189219504514 0 rpy=0 0 0
- joint j4: origin xyz=0 0.47119707676675754 0.0203999999999699 rpy=1.57079632675385 0 -3.14159265356591 -> xyz=0 0.23745357169153747 0.0203999999999699 rpy=1.57079632675385 0 -3.14159265356591

Commit message: fixed ddqn tested-model

File: dynamics/src/dynamics/urdf/random.urdf (robot description, URDF)
Before this commit: robot tecobot, 8 links, 7 joints
Links:
- link 2: mass 1.7679247444870383 -> 1.7091452845402997
- link 3: mass 0.4721316268780683 -> 0.5226810145479754
Joints:
- joint j3: origin xyz=0 0.4836189219504514 0 rpy=0 0 0 -> xyz=0 0.31135179187490003 0 rpy=0 0 0
- joint j4: origin xyz=0 0.23745357169153747 0.0203999999999699 rpy=1.57079632675385 0 -3.14159265356591 -> xyz=0 0.3856005255570863 0.0203999999999699 rpy=1.57079632675385 0 -3.14159265356591

Commit message: add manipulability method

File: dynamics/src/dynamics/urdf/random.urdf (robot description, URDF)
Before this commit: robot tecobot, 8 links, 7 joints
Links:
- link 2: mass 1.7091452845402997 -> 1.7351088174173208
- link 3: mass 0.5226810145479754 -> 0.5159966584840698
Joints:
- joint j3: origin xyz=0 0.31135179187490003 0 rpy=0 0 0 -> xyz=0 0.38744407478119824 0 rpy=0 0 0
- joint j4: origin xyz=0 0.3856005255570863 0.0203999999999699 rpy=1.57079632675385 0 -3.14159265356591 -> xyz=0 0.3660104368326318 0.0203999999999699 rpy=1.57079632675385 0 -3.14159265356591

Commit message: add reach_score & manipulability_score

File: dynamics/src/dynamics/urdf/random.urdf (robot description, URDF)
Before this commit: robot tecobot, 8 links, 7 joints
Links:
- link 2: mass 1.7351088174173208 -> 1.754493177881885
- link 3: mass 0.5159966584840698 -> 0.5218924164974693
Joints:
- joint j3: origin xyz=0 0.38744407478119824 0 rpy=0 0 0 -> xyz=0 0.4442545345677671 0 rpy=0 0 0
- joint j4: origin xyz=0 0.3660104368326318 0.0203999999999699 rpy=1.57079632675385 0 -3.14159265356591 -> xyz=0 0.38328935218007737 0.0203999999999699 rpy=1.57079632675385 0 -3.14159265356591

Commit message: add reach & manipulability & fixed reward function

File: dynamics/src/dynamics/urdf/random.urdf (robot description, URDF)
Before this commit: robot tecobot, 8 links, 7 joints
Links:
- link 2: mass 1.754493177881885 -> 1.7358726479243753
- link 3: mass 0.5218924164974693 -> 0.5220871289582969
Joints:
- joint j3: origin xyz=0 0.4442545345677671 0 rpy=0 0 0 -> xyz=0 0.3896826610055979 0 rpy=0 0 0
- joint j4: origin xyz=0 0.38328935218007737 0.0203999999999699 rpy=1.57079632675385 0 -3.14159265356591 -> xyz=0 0.3838600031667843 0.0203999999999699 rpy=1.57079632675385 0 -3.14159265356591

Commit message: fixed self.state[9] = manipulability_score

File: dynamics/src/dynamics/urdf/random.urdf (robot description, URDF)
Before this commit: robot tecobot, 8 links, 7 joints
Links:
- link 2: mass 1.7358726479243753 -> 1.6756116446037903
- link 3: mass 0.5220871289582969 -> 0.5572653264164609
Joints:
- joint j3: origin xyz=0 0.3896826610055979 0 rpy=0 0 0 -> xyz=0 0.21307351714961667 0 rpy=0 0 0
- joint j4: origin xyz=0 0.3838600031667843 0.0203999999999699 rpy=1.57079632675385 0 -3.14159265356591 -> xyz=0 0.4869580432447316 0.0203999999999699 rpy=1.57079632675385 0 -3.14159265356591

Commit message: TODO: fixed 0112 00:22

File: dynamics/src/dynamics/urdf/random.urdf (robot description, URDF)
Before this commit: robot tecobot, 8 links, 7 joints
Links:
- link 2: mass 1.6756116446037903 -> 1.7399207547798456
- link 3: mass 0.5572653264164609 -> 0.5031298859074359
Joints:
- joint j3: origin xyz=0 0.21307351714961667 0 rpy=0 0 0 -> xyz=0 0.40154659699383133 0 rpy=0 0 0
- joint j4: origin xyz=0 0.4869580432447316 0.0203999999999699 rpy=1.57079632675385 0 -3.14159265356591 -> xyz=0 0.32830131212954716 0.0203999999999699 rpy=1.57079632675385 0 -3.14159265356591

Commit message: TODO: fixed reward function

File: dynamics/src/dynamics/urdf/random.urdf (robot description, URDF)
Before this commit: robot tecobot, 8 links, 7 joints
Links:
- link 2: mass 1.7399207547798456 -> 1.7669762476910225
- link 3: mass 0.5031298859074359 -> 0.49801879403681754
Joints:
- joint j3: origin xyz=0 0.40154659699383133 0 rpy=0 0 0 -> xyz=0 0.48083912742556806 0 rpy=0 0 0
- joint j4: origin xyz=0 0.32830131212954716 0.0203999999999699 rpy=1.57079632675385 0 -3.14159265356591 -> xyz=0 0.3133220467721975 0.0203999999999699 rpy=1.57079632675385 0 -3.14159265356591

Commit message: fixed reward shape

File: dynamics/src/dynamics/urdf/random.urdf (robot description, URDF)
Before this commit: robot tecobot, 8 links, 7 joints
Links:
- link 2: mass 1.7669762476910225 -> 1.7353705512263176
- link 3: mass 0.49801879403681754 -> 0.5132181299796656
Joints:
- joint j3: origin xyz=0 0.48083912742556806 0 rpy=0 0 0 -> xyz=0 0.38821114770361803 0 rpy=0 0 0
- joint j4: origin xyz=0 0.3133220467721975 0.0203999999999699 rpy=1.57079632675385 0 -3.14159265356591 -> xyz=0 0.35786730091881863 0.0203999999999699 rpy=1.57079632675385 0 -3.14159265356591

Commit message: aa

File: dynamics/src/dynamics/urdf/random.urdf (robot description, URDF)
Before this commit: robot tecobot, 8 links, 7 joints
Links:
- link 2: mass 1.7353705512263176 -> 1.6508092151221665
- link 3: mass 0.5132181299796656 -> 0.4964628887269289
Joints:
- joint j3: origin xyz=0 0.38821114770361803 0 rpy=0 0 0 -> xyz=0 0.14038412276640627 0 rpy=0 0 0
- joint j4: origin xyz=0 0.35786730091881863 0.0203999999999699 rpy=1.57079632675385 0 -3.14159265356591 -> xyz=0 0.3087620977245759 0.0203999999999699 rpy=1.57079632675385 0 -3.14159265356591
